Commit message: odom test

File: src/serial_comm/serial_comm/robot_description.urdf (robot description, URDF)
Before this commit: robot amr, 8 links, 7 joints
Joints:
- joint base_joint: origin xyz=0 0 0.2175 rpy=0 0 3.14 -> xyz=0 0 0.2175 rpy=0 0 0
- joint wheel_left_joint: origin xyz=-0.14 0.16 -0.1425 rpy=3.14 0 0 -> xyz=-0.14 0.16 -0.1425 rpy=0 0 0
- joint wheel_right_joint: origin xyz=-0.14 -0.16 -0.1425 rpy=3.14 0 0 -> xyz=-0.14 -0.16 -0.1425 rpy=0 0 0
