Commit message: urdf test

File: src/robot_description/description/robot_description.urdf (robot description, URDF)
Before this commit: robot amr, 15 links, 14 joints
Links:
- removed link caster_back_left_link
- removed link caster_back_right_link
- removed link caster_front_left_link
- removed link caster_front_right_link
- removed link caster_wheel_back_left_link
- removed link caster_wheel_back_right_link
- removed link caster_wheel_front_left_link
- removed link caster_wheel_front_right_link
- link wheel_left_link: geometry collision cylinder length=0.046 radius=0.065; visual mesh filename=package://amr_demo/description/meshes/amr_wheel.stl scale=0.001 0.001 0.001
- link wheel_right_link: geometry collision cylinder length=0.046 radius=0.065; visual mesh filename=package://amr_demo/description/meshes/amr_wheel.stl scale=0.001 0.001 0.001
Joints:
- removed joint caster_back_left_joint
- removed joint caster_back_right_joint
- removed joint caster_front_left_joint
- removed joint caster_front_right_joint
- removed joint caster_wheel_back_left_joint
- removed joint caster_wheel_back_right_joint
- removed joint caster_wheel_front_left_joint
- removed joint caster_wheel_front_right_joint
- joint lidar1_joint: origin xyz=0.24698 0.143555 0.2 rpy=0. 0 -1.57 -> xyz=0.105 -0.075 0.25 rpy=0 0 0
- joint lidar2_joint: origin xyz=-0.24698 -0.143555 0.2 rpy=0. 0 1.57 -> xyz=-0.105 0.075 0.25 rpy=0 0 3.14159
- joint lidar_joint: origin xyz=0.0 0.0 0.2 rpy=0 0 -1.57 -> xyz=0.0 0.0 0.0 rpy=0 0 0
- joint wheel_left_joint: origin xyz=0 0.145 0.085 rpy=-1.57 0 0 -> xyz=0 0.16 -0.065 rpy=-1.57 0 0
- joint wheel_right_joint: origin xyz=0 -0.145 0.085 rpy=1.57 0 0 -> xyz=0 -0.16 -0.065 rpy=1.57 0 0

Commit message: tf logic update

File: src/robot_description/description/robot_description.urdf (robot description, URDF)
Before this commit: robot amr, 7 links, 6 joints
Joints:
- joint wheel_left_joint: axis (none) -> 0 1 0; type fixed -> continuous
- joint wheel_right_joint: axis (none) -> 0 1 0; type fixed -> continuous

Commit message: urdf test

File: src/robot_description/description/robot_description.urdf (robot description, URDF)
Before this commit: robot amr, 7 links, 6 joints
Links:
- link chassis: mass 1.37291 -> None; geometry visual box size=0.30 0.25 0.215
- link laser: mass 0.114 -> None
- link lidar1_link: mass 0.114 -> None
- link lidar2_link: mass 0.114 -> None
- link wheel_left_link: mass 0.1 -> None; geometry visual cylinder length=0.065 radius=0.065
- link wheel_right_link: mass 0.1 -> None; geometry visual cylinder length=0.065 radius=0.065
Joints:
- joint base_joint: origin xyz=0 0 0.001 rpy=0 0 0 -> xyz=0 0 0.2175 rpy=0 0 0
- joint lidar1_joint: origin xyz=0.105 -0.075 0.25 rpy=0 0 0 -> xyz=0.105 -0.075 0.13 rpy=0 0 0
- joint lidar2_joint: origin xyz=-0.105 0.075 0.25 rpy=0 0 3.14159 -> xyz=-0.105 0.075 0.13 rpy=0 0 3.14159
- joint lidar_joint: origin xyz=0.0 0.0 0.0 rpy=0 0 0 -> xyz=0.0 0.0 0.13 rpy=0 0 0
- joint wheel_left_joint: origin xyz=0 0.16 -0.065 rpy=-1.57 0 0 -> xyz=0.14 0.16 -0.1425 rpy=-1.57 0 0
- joint wheel_right_joint: origin xyz=0 -0.16 -0.065 rpy=1.57 0 0 -> xyz=0.14 -0.16 -0.1425 rpy=1.57 0 0

Commit message: TEST

File: src/robot_description/description/robot_description.urdf (robot description, URDF)
Before this commit: robot amr, 7 links, 6 joints
Joints:
- joint wheel_left_joint: origin xyz=0.14 0.16 -0.1425 rpy=-1.57 0 0 -> xyz=0.14 0.16 -0.1425 rpy=0 0 0
- joint wheel_right_joint: origin xyz=0.14 -0.16 -0.1425 rpy=1.57 0 0 -> xyz=0.14 -0.16 -0.1425 rpy=0 0 0

Commit message: desc, base main update

File: src/robot_description/description/robot_description.urdf (robot description, URDF)
Before this commit: robot amr, 7 links, 6 joints
Joints:
- joint wheel_left_joint: origin xyz=0.14 0.16 -0.1425 rpy=0 0 0 -> xyz=-0.14 0.16 -0.1425 rpy=0 0 0
- joint wheel_right_joint: origin xyz=0.14 -0.16 -0.1425 rpy=0 0 0 -> xyz=-0.14 -0.16 -0.1425 rpy=0 0 0

Commit message: test

File: src/robot_description/description/robot_description.urdf (robot description, URDF)
Before this commit: robot amr, 7 links, 6 joints
Links:
- added link imu_link; visual box size=0.02 0.02 0.01
Joints:
- added joint imu_joint: type fixed, parent chassis, child imu_link, origin xyz=-0.03 0.0 0.0 rpy=0 0 0

Commit message: odom finish

File: src/robot_description/description/robot_description.urdf (robot description, URDF)
Before this commit: robot amr, 8 links, 7 joints
Joints:
- joint base_joint: origin xyz=0 0 0.2175 rpy=0 0 3.14 -> xyz=0 0 0.2175 rpy=0 0 0
- joint lidar_joint: origin xyz=0.0 0.0 0.13 rpy=0 0 0 -> xyz=0.0 0.0 0.13 rpy=0 0 3.14
- joint wheel_left_joint: axis 0 1 0 -> 0 -1 0; origin xyz=-0.14 0.16 -0.1425 rpy=3.14 0 0 -> xyz=-0.14 0.16 -0.1425 rpy=0 0 0
- joint wheel_right_joint: axis 0 1 0 -> 0 -1 0; origin xyz=-0.14 -0.16 -0.1425 rpy=3.14 0 0 -> xyz=-0.14 -0.16 -0.1425 rpy=0 0 0

Commit message: robot description update(final)

File: src/robot_description/description/robot_description.urdf (robot description, URDF)
Before this commit: robot amr, 8 links, 7 joints
Joints:
- joint wheel_left_joint: origin xyz=-0.14 0.16 -0.1425 rpy=0 0 0 -> xyz=0.14 0.16 -0.1425 rpy=0 0 0
- joint wheel_right_joint: origin xyz=-0.14 -0.16 -0.1425 rpy=0 0 0 -> xyz=0.14 -0.16 -0.1425 rpy=0 0 0
